Commit message: mybot_apps

File: src/mybot_bringup/urdf/mybot.urdf.xacro (robot description, xacro)
@@ -3,5 +3,5 @@
   <!-- Ajuste esses valores -->
   <xacro:property name="wheel_radius" value="0.0325"/>
-  <xacro:property name="wheel_separation" value="0.158"/>
+  <xacro:property name="wheel_separation" value="0.155"/>
   <link name="base_link"/>
   <link name="left_wheel_link"/>

Commit message: calibration tests

File: src/mybot_bringup/urdf/mybot.urdf.xacro (robot description, xacro)
@@ -2,5 +2,5 @@
 <robot name="mybot" xmlns:xacro="http://www.ros.org/wiki/xacro">
   <!-- Ajuste esses valores -->
-  <xacro:property name="wheel_radius" value="0.0325"/>
+  <xacro:property name="wheel_radius" value="0.03187"/>
   <xacro:property name="wheel_separation" value="0.155"/>
   <link name="base_link"/>
